Commit message: Standard properties

File: robot.urdf.xacro (robot description, xacro)
@@ -18,5 +18,5 @@
     <xacro:property name="chassis_head" value="0.473"/>
     <xacro:property name="chassis_tail" value="0.473"/>
-    <xacro:property name="chassis_width" value="0.8"/>
+    <xacro:property name="chassis_width" value="0.685"/>
     <xacro:property name="chassis_height" value="0.3"/>
     <xacro:property name="chassis_z" value="0.102"/>
@@ -39,6 +39,6 @@
     <xacro:property name="right_wheel_thickness" value="0.05"/>
     <xacro:property name="right_wheel_sign" value="-1"/>
-    <xacro:property name="lidar_1_x" value="0.2"/>
-    <xacro:property name="lidar_1_y" value="0.2"/>
+    <xacro:property name="lidar_1_x" value="0.45"/>
+    <xacro:property name="lidar_1_y" value="0.3"/>
     <xacro:property name="lidar_1_z" value="0.41"/>
     <xacro:property name="lidar_1_roll" value="0.0"/>
